File: electronics/OpenESPTemp.kicad_sch (KiCad schematic)
At the start: 42 parts, among them J2 Qwiic_RA, Q1 TSM260P02CX-RFG, Q2 DMN2020LSN-7, SW1 WAKE, SW2 FCT, SW3 BOOT, SW4 RESET, U2 RV-3028-C7, U3 BME280, U4 TLV70033_SOT23-5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

Commit message: Fix Pcb issues
- Fix wrong connection of C4
- Move symbol lib into libs/; Delete unused .kicad_sch file
- Make LDO Solder Jumper Bridged by default
- Fix temp notes file (Licenses.txt)
Parts:
- JP2: footprint Jumper:SolderJumper-2_P1.3mm_Open_RoundedPad1.0x1.5mm -> Jumper:SolderJumper-2_P1.3mm_Bridged_RoundedPad1.0x1.5mm; symbol Jumper:SolderJumper_2_Open -> Jumper:SolderJumper_2_Bridged
Connections:
- net +BATT: now also C4.1, U2.7 (VDD); no longer C4.2
- net GND: now also C4.2
Other:
- note removed: "3v3 or BATT?"

Commit message: fix(electronics): Improve Schematic
Improve schematic overall
Add exported .pdf of current schematics
Connections:
- net +3V3: now also R6.1; no longer R6.2
- net SDA: now also R6.2; no longer R6.1
Other:
- moved on the sheet: J2, R2, R5, R6
